File: capstone/capstone.kicad_sch (KiCad schematic)
At the start: 16 parts, among them J1 Conn_01x02, M1 Motor_Servo, M2 Motor_Servo, M3 Stepper_Motor_bipolar, M4 Stepper_Motor_bipolar, SW1 SW_Push, U1 PicoW

Commit message: remove 12v regulators + pcb traces
Parts:
- removed PWR_regulator1, PWR_regulator2: ~, capstone:YAAJ_DCDC_StepDown_LM2596, symbol New_Library:Power_regulator
Connections:
- net Servo_PWR_5V is gone; now on net PICO_PWR_5V: M1.2 (+), M2.2 (+)
- net Stepper_PWR_12V is gone; now on net 14V: A1.8 (VMOT), A2.8 (VMOT), C1.1, C2.1
- net Lipo renamed 14V
- net VBUS: no longer names the net of U1.40 (VBUS)
- no-connect marks 19 -> 20
Other:
- moved on the sheet: IR_sensor1, IR_sensor2, J1, M1, M2, M3, M4, PWR_regulator3
